File: Schörkhuber/KiCAD/BLDC_Motor_neu_1/BLDC_Motor_neu_1.kicad_pcb (KiCad board)
At the start: 2 copper layers, 104.8 x 38.7 mm, 30 parts, among them J1 Conn_01x03_Pin, J2 Conn_01x01, J3 Conn_01x01, J4 Conn_01x01, Q1 DMN3042L, Q2 DMN3042L, Q3 DMP3099L, Q4 DMN3042L, Q5 DMN3042L, Q6 DMP3099L, Q7 DMN3042L, Q8 DMN3042L, Q9 DMP3099L, U1 Waveshare-RP2040-Zero

Commit message: AUfgaben
Parts:
- moved R25 1.91 mm to (152.8, 95.9)
Routing:
- net Net-(U1-GP3): track 42.6 -> 43.6 mm
- net Net-(J1-Pin_2): track 20.9 -> 21.5 mm
